File: Project/Eightu Ortho.kicad_pcb (KiCad board)
At the start: 2 copper layers, 250.9 x 79.4 mm, 141 parts, among them J1 JST SH, J2 Pico EZmate, SW1 RotaryEncoder_Switch, SW2 RotaryEncoder_Switch, SW3 RotaryEncoder_Switch, SW4 RotaryEncoder_Switch, SW5 RotaryEncoder_Switch, SW6 SKQGABE010, SW7 RotaryEncoder_Switch, U1 STM32F072CBT6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

Commit message: fresh ortho gerbers
Routing:
- net GND: track 36.2 -> 50.7 mm, vias 9 -> 15
