File: Project/Eightu.kicad_pcb (KiCad board)
At the start: 2 copper layers, 250.9 x 79.4 mm, 134 parts, among them J1 JST SH, J2 Pico EZmate, SW1 RotaryEncoder_Switch, SW2 RotaryEncoder_Switch, SW3 RotaryEncoder_Switch, SW4 RotaryEncoder_Switch, SW5 RotaryEncoder_Switch, SW6 SKQGABE010, U1 STM32F072CBT6, U2 XC6206PxxxMR-Regulator_Linear

Commit message: firmware update
Routing:
- net GND: track 36.2 -> 36.1 mm, vias 9 -> 13
Changed lines of the file:
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@@
     (fp_arc (start 8.53125 -5.499999) (mid 8.677685 -5.853565) (end 9.03125 -5.999999)
       (stroke (width 0.05) (type solid)) (layer "Eco2.User"))
-    (fp_arc (start 9.03125 8.000001) (mid 8.677693 7.853543) (end 8.53125 7.500001)
+    (fp_arc (start 9.03125 8.000001) (mid 8.677729 7.853537) (end 8.53125 7.500001)
       (stroke (width 0.05) (type solid)) (layer "Eco2.User"))
-    (fp_arc (start 14.780039 -5.999999) (mid 15.133602 -5.853545) (end 15.280039 -5.499999)
+    (fp_arc (start 14.780039 -5.999999) (mid 15.133567 -5.853539) (end 15.280039 -5.499999)
       (stroke (width 0.05) (type solid)) (layer "Eco2.User"))
-    (fp_arc (start 15.28125 7.500001) (mid 15.1348 7.853536) (end 14.78125 8.000001)
+    (fp_arc (start 15.28125 7.500001) (mid 15.134806 7.853571) (end 14.78125 8.000001)
       (stroke (width 0.05) (type solid)) (layer "Eco2.User"))
     (pad "" thru_hole circle (at -11.90625 -6.985 180) (size 4 4) (drill 3.048) (layers "*.Cu" "B.Mask"))
@@
     (fp_arc (start 8.53125 -5.499999) (mid 8.677685 -5.853565) (end 9.03125 -5.999999)
       (stroke (width 0.05) (type solid)) (layer "Eco2.User"))
-    (fp_arc (start 9.03125 8.000001) (mid 8.677729 7.853537) (end 8.53125 7.500001)
+    (fp_arc (start 9.03125 8.000001) (mid 8.677693 7.853543) (end 8.53125 7.500001)
       (stroke (width 0.05) (type solid)) (layer "Eco2.User"))
-    (fp_arc (start 14.780039 -5.999999) (mid 15.133567 -5.853539) (end 15.280039 -5.499999)
+    (fp_arc (start 14.780039 -5.999999) (mid 15.133602 -5.853545) (end 15.280039 -5.499999)
       (stroke (width 0.05) (type solid)) (layer "Eco2.User"))
-    (fp_arc (start 15.28125 7.500001) (mid 15.134806 7.853571) (end 14.78125 8.000001)
+    (fp_arc (start 15.28125 7.500001) (mid 15.1348 7.853536) (end 14.78125 8.000001)
       (stroke (width 0.05) (type solid)) (layer "Eco2.User"))
     (pad "" thru_hole circle (at -11.90625 -6.985 180) (size 4 4) (drill 3.048) (layers "*.Cu" "B.Mask"))
@@
     (fp_arc (start 8.53125 -5.499999) (mid 8.677685 -5.853565) (end 9.03125 -5.999999)
       (stroke (width 0.05) (type solid)) (layer "Eco2.User"))
-    (fp_arc (start 9.03125 8.000001) (mid 8.677693 7.853543) (end 8.53125 7.500001)
+    (fp_arc (start 9.03125 8.000001) (mid 8.677729 7.853537) (end 8.53125 7.500001)
       (stroke (width 0.05) (type solid)) (layer "Eco2.User"))
-    (fp_arc (start 14.780039 -5.999999) (mid 15.133602 -5.853545) (end 15.280039 -5.499999)
+    (fp_arc (start 14.780039 -5.999999) (mid 15.133567 -5.853539) (end 15.280039 -5.499999)
       (stroke (width 0.05) (type solid)) (layer "Eco2.User"))
-    (fp_arc (start 15.28125 7.500001) (mid 15.1348 7.853536) (end 14.78125 8.000001)
+    (fp_arc (start 15.28125 7.500001) (mid 15.134806 7.853571) (end 14.78125 8.000001)
       (stroke (width 0.05) (type solid)) (layer "Eco2.User"))
     (pad "" thru_hole circle (at -11.90625 -6.985 180) (size 4 4) (drill 3.048) (layers "*.Cu" "B.Mask"))
@@
     (fp_arc (start 8.53125 -5.499999) (mid 8.677685 -5.853565) (end 9.03125 -5.999999)
       (stroke (width 0.05) (type solid)) (layer "Eco2.User"))
-    (fp_arc (start 9.03125 8.000001) (mid 8.677729 7.853537) (end 8.53125 7.500001)
+    (fp_arc (start 9.03125 8.000001) (mid 8.677693 7.853543) (end 8.53125 7.500001)
       (stroke (width 0.05) (type solid)) (layer "Eco2.User"))
-    (fp_arc (start 14.780039 -5.999999) (mid 15.133567 -5.853539) (end 15.280039 -5.499999)
+    (fp_arc (start 14.780039 -5.999999) (mid 15.133602 -5.853545) (end 15.280039 -5.499999)
       (stroke (width 0.05) (type solid)) (layer "Eco2.User"))
-    (fp_arc (start 15.28125 7.500001) (mid 15.134806 7.853571) (end 14.78125 8.000001)
+    (fp_arc (start 15.28125 7.500001) (mid 15.1348 7.853536) (end 14.78125 8.000001)
       (stroke (width 0.05) (type solid)) (layer "Eco2.User"))
     (pad "" thru_hole circle (at -11.90625 -6.985 180) (size 4 4) (drill 3.048) (layers "*.Cu" "B.Mask"))
@@
   (segment (start 296.1875 59.8875) (end 297.0625 59.0125) (width 0.25) (layer "B.Cu") (net 65))
   (segment (start 290.452271 77.1625) (end 289.564771 78.05) (width 0.25) (layer "B.Cu") (net 65))
+  (via (at 282.74447 76.549972) (size 0.8) (drill 0.4) (layers "F.Cu" "B.Cu") (net 66))
+  (via (at 276.762718 89.171339) (size 0.8) (drill 0.4) (layers "F.Cu" "B.Cu") (net 66))
   (via (at 280.90387 66.314604) (size 0.8) (drill 0.4) (layers "F.Cu" "B.Cu") (net 66))
   (via (at 282.575 69.85) (size 0.8) (drill 0.4) (layers "F.Cu" "B.Cu") (net 66))
@@
   (via (at 269.875 76.2) (size 0.8) (drill 0.4) (layers "F.Cu" "B.Cu") (net 66))
   (via (at 279.995956 63.374119) (size 0.8) (drill 0.4) (layers "F.Cu" "B.Cu") (net 66))
+  (via (at 284.87432 83.475232) (size 0.8) (drill 0.4) (layers "F.Cu" "B.Cu") (net 66))
   (via (at 277.01875 80.3) (size 0.8) (drill 0.4) (layers "F.Cu" "B.Cu") (net 66))
-  (via (at 276.224893 89.176406) (size 0.8) (drill 0.4) (layers "F.Cu" "B.Cu") (net 66))
+  (via (at 280.91069 71.4375) (size 0.8) (drill 0.4) (layers "F.Cu" "B.Cu") (net 66))
   (via (at 254.175142 61.02074) (size 0.8) (drill 0.4) (layers "F.Cu" "B.Cu") (net 66))
+  (via (at 275.769317 89.161098) (size 0.8) (drill 0.4) (layers "F.Cu" "B.Cu") (net 66))
   (segment (start 279.26875 82.55) (end 277.01875 80.3) (width 0.25) (layer "B.Cu") (net 66))
   (segment (start 281.18125 82.55) (end 279.26875 82.55) (width 0.25) (layer "B.Cu") (net 66))
+  (segment (start 282.751298 76.543144) (end 282.74447 76.549972) (width 0.381) (layer "B.Cu") (net 66))
+  (segment (start 276.765057 88.238459) (end 276.765057 89.169) (width 0.25) (layer "B.Cu") (net 66))
   (segment (start 276.26875 81.05) (end 277.01875 80.3) (width 0.25) (layer "B.Cu") (net 66))
   (segment (start 283.769189 84.761185) (end 283.778293 84.752081) (width 0.381) (layer "B.Cu") (net 66))
-  (segment (start 282.751298 74.738798) (end 282.751298 75.7375) (width 0.381) (layer "B.Cu") (net 66))
-  (segment (start 276.225 89.176299) (end 276.224893 89.176406) (width 0.381) (layer "B.Cu") (net 66))
+  (segment (start 275.768435 89.160216) (end 275.769317 89.161098) (width 0.25) (layer "B.Cu") (net 66))
   (segment (start 274.76875 78.05) (end 277.01875 80.3) (width 0.25) (layer "B.Cu") (net 66))
-  (segment (start 276.764098 88.2375) (end 276.765057 88.238459) (width 0.381) (layer "B.Cu") (net 66))
+  (segment (start 284.874088 83.475) (end 284.87432 83.475232) (width 0.381) (layer "B.Cu") (net 66))
   (segment (start 251.985197 60.4125) (end 252.825 60.4125) (width 0.381) (layer "B.Cu") (net 66))
   (segment (start 280.90282 66.315654) (end 280.90387 66.314604) (width 0.25) (layer "B.Cu") (net 66))
   (segment (start 276.26875 84.4625) (end 276.26875 81.05) (width 0.25) (layer "B.Cu") (net 66))
-  (segment (start 276.225 88.2375) (end 276.764098 88.2375) (width 0.381) (layer "B.Cu") (net 66))
   (segment (start 281.14375 69.85) (end 282.575 69.85) (width 0.25) (layer "B.Cu") (net 66))
+  (segment (start 279.99 71.4375) (end 280.91069 71.4375) (width 0.25) (layer "B.Cu") (net 66))
+  (segment (start 282.751298 75.7375) (end 282.751298 76.543144) (width 0.381) (layer "B.Cu") (net 66))
   (segment (start 279.999995 62.376265) (end 279.999995 63.37008) (width 0.25) (layer "B.Cu") (net 66))
   (segment (start 271.0025 76.2) (end 269.875 76.2) (width 0.381) (layer "B.Cu") (net 66))
@@
   (segment (start 279.99 66.315654) (end 280.90282 66.315654) (width 0.25) (layer "B.Cu") (net 66))
   (segment (start 272.85625 78.05) (end 274.76875 78.05) (width 0.25) (layer "B.Cu") (net 66))
-  (segment (start 275.768435 88.2375) (end 276.225 88.2375) (width 0.381) (layer "B.Cu") (net 66))
   (segment (start 247.910197 58.9625) (end 248.8 58.9625) (width 0.25) (layer "B.Cu") (net 66))
   (segment (start 279.26875 78.05) (end 277.01875 80.3) (width 0.25) (layer "B.Cu") (net 66))
   (segment (start 252.825 60.4125) (end 253.566902 60.4125) (width 0.381) (layer "B.Cu") (net 66))
+  (segment (start 275.768435 88.2375) (end 275.768435 89.160216) (width 0.25) (layer "B.Cu") (net 66))
   (segment (start 253.566902 60.4125) (end 254.175142 61.02074) (width 0.381) (layer "B.Cu") (net 66))
   (segment (start 281.9625 73.95) (end 282.751298 74.738798) (width 0.381) (layer "B.Cu") (net 66))
   (segment (start 282.810882 84.761185) (end 282.751298 84.761185) (width 0.381) (layer "B.Cu") (net 66))
+  (segment (start 283.996827 83.475) (end 284.874088 83.475) (width 0.381) (layer "B.Cu") (net 66))
   (segment (start 247.910197 64.8625) (end 248.8 64.8625) (width 0.25) (layer "B.Cu") (net 66))
-  (segment (start 283.996827 83.57524) (end 282.810882 84.761185) (width 0.381) (layer "B.Cu") (net 66))
+  (segment (start 276.765057 89.169) (end 276.762718 89.171339) (width 0.25) (layer "B.Cu") (net 66))
   (segment (start 279.26875 76.1375) (end 279.26875 78.05) (width 0.25) (layer "B.Cu") (net 66))
   (segment (start 248.8 64.8625) (end 248.95 64.7125) (width 0.25) (layer "B.Cu") (net 66))
   (segment (start 283.996827 83.475) (end 283.996827 83.57524) (width 0.381) (layer "B.Cu") (net 66))
-  (segment (start 276.225 88.2375) (end 276.225 89.176299) (width 0.381) (layer "B.Cu") (net 66))
   (segment (start 282.751298 84.761185) (end 283.769189 84.761185) (width 0.381) (layer "B.Cu") (net 66))
   (segment (start 291.1875 78.9375) (end 291.075 79.05) (width 0.25) (layer "B.Cu") (net 67))

Commit message: update gerbers
Routing:
- net GND: track 36.1 -> 46.8 mm, vias 13 -> 18
